File: basketweave/basketweave.kicad_pcb (KiCad board)
At the start: 2 copper layers, 371.5 x 145.3 mm, 177 parts, among them J1 AVR-ISP-6, SW1 SW_Push, SW2 SW_Push, SW3 Rotary_Encoder_Switch, U1 ATmega32A-PU, U2 GCT-USB-4085-GF-A, Y1 16Mhz

Commit message: Make macro keys symmetric on both sides; move encoder to the left
Parts:
- added MX16: MX-NoLED, MX_Only:MXOnly-1U-NoLED, F.Cu at (42.1, 134.9)
- added MX75: MX-NoLED, MX_Only:MXOnly-1U-NoLED, F.Cu at (37.3, 154.0)
- moved SW3 11.5 mm to (39.8, 146.5), turned to 270 degrees
- moved D72 0.06 mm to (366.8, 124.2)
Connections:
- D16 pad 2: (no net) -> Net-(D16-Pad2)
- U2 pad B1: Net-(U2-PadB1) -> GND
- U2 pad S1: Net-(U2-PadB1) -> GND
Routing:
- net GND: track 97.3 -> 26.2 mm, vias 7 -> 8
- net Net-(D16-Pad2): track 0.00 -> 41.1 mm
- net EN2: track 236.1 -> 221.7 mm
- net Net-(D31-Pad2): track 64.8 -> 73.5 mm
- net COL0: track 186.6 -> 193.1 mm
- net EN1: track 226.7 -> 222.8 mm
Other:
- board text added: "Basketweave-S"
- board text added: "Modified by piit79"
- board text added: "Rev 1.5"
- board text added: "github.com/piit79/basketweave-s"
- board text removed: "Rev 1"
