File: basketweave_bottom/basketweave_bottom.kicad_pcb (KiCad board)
At the start: 2 copper layers, 371.5 x 145.3 mm, 14 parts

Commit message: Make macro keys symmetric on both sides; move encoder to the left
Parts:
- moved H2 1.13 mm to (27.0, 94.4)
- moved H4 1.13 mm to (390.5, 94.4)
- moved H5 0.83 mm to (161.8, 94.4)
- moved H6 0.83 mm to (231.9, 94.4)
- moved H1 0.76 mm to (27.0, 77.0)
- moved H3 0.76 mm to (390.5, 77.0)

Commit message: Modify bottom plate logo for Basketweave-S and move it into PCB footprint library
Parts:
- removed the G*** at (205.6, 140.5)
- added G***: LOGO, basketweave:logo_bottom, B.Cu at (220.1, 140.3)
Other:
- board text added: "JLCJLCJLCJLC"
